File: OdD1/untitled.sch (EAGLE design)
At the start: 9 parts, among them U1 74HC4052DIP, U2 ATMEGA328P-PU, U3 74HC4052DIP, U4 74HC4052DIP, U5 74HC4052DIP, U6 74HC4052DIP, U7 74HC4052DIP

Commit message: Change counter reset pin. Need to set pin directions first
Connections:
- new net MCU_RST: U2.PC6
- net ADC_RST: now also U2.PD7; no longer U2.PC6
Changed lines of the file:
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@@
 </segment>
 <segment>
-<pinref part="U2" gate="A" pin="PC6"/>
-<wire x1="93.98" y1="55.88" x2="116.84" y2="55.88" width="0.1524" layer="91"/>
-<label x="96.52" y="55.88" size="1.778" layer="95"/>
+<pinref part="U2" gate="A" pin="PD7"/>
+<wire x1="93.98" y1="76.2" x2="109.22" y2="76.2" width="0.1524" layer="91"/>
+<label x="96.52" y="76.2" size="1.778" layer="95"/>
 </segment>
 </net>
@@
 </segment>
 </net>
+<net name="MCU_RST" class="0">
+<segment>
+<pinref part="U2" gate="A" pin="PC6"/>
+<wire x1="93.98" y1="55.88" x2="116.84" y2="55.88" width="0.1524" layer="91"/>
+<label x="96.52" y="55.88" size="1.778" layer="95"/>
+</segment>
+</net>
